Commit message: wip: update moveit config for stretch robotiq robot

File: stretch_robotiq_moveit_config/config/gazebo_stretch.urdf (robot description, URDF)
Before this commit: robot stretch, 48 links, 47 joints
Links:
- added link link_grasp_center
Joints:
- added joint joint_grasp_center: type fixed, parent robotiq_arg2f_base_link, child link_grasp_center, origin xyz=0 0 0.2 rpy=0 0 0
