Commit message: wip: use link_grasp_center as streach_arm planning frame

File: stretch_robotiq_description/urdf/stretch_robotiq_description.xacro (robot description, xacro)
@@ -20,4 +20,10 @@
       xyz="0 0 0" />
   </joint>
+  <link name="link_grasp_center" />
+  <joint name="joint_grasp_center" type="fixed">
+      <origin rpy="0 0 0" xyz="0 0 0.2" />
+      <parent link="robotiq_arg2f_base_link" />
+      <child link="link_grasp_center" />
+  </joint>
   <xacro:include filename="stretch_main.xacro" />
   <xacro:include filename="stretch_aruco.xacro" />
