Commit message: wip: update missing link_grasp_center and base_imu frames

File: stretch_gazebo/urdf/stretch_robotiq_gazebo.urdf.xacro (robot description, xacro)
@@ -8,4 +8,5 @@
   <xacro:include filename="$(find stretch_gazebo)/urdf/stretch_laser_range_finder.xacro" />
   <xacro:include filename="$(find stretch_gazebo)/urdf/stretch_respeaker.xacro" />
+  <xacro:include filename="$(find stretch_gazebo)/urdf/stretch_base_imu.xacro" />
   <xacro:include filename="$(find robotiq_2f_140_gripper_visualization)/urdf/robotiq_arg2f_140_model.xacro" />
   <!-- <xacro:include filename="$(find stretch_robotiq_description)/urdf/robotiq_arg85_description.xacro" /> -->
@@ -502,4 +503,10 @@
     <axis
       xyz="0 0 0" />
+  </joint>
+  <link name="link_grasp_center" />
+  <joint name="joint_grasp_center" type="fixed">
+      <origin rpy="0 0 0" xyz="0 0 0.2" />
+      <parent link="robotiq_arg2f_base_link" />
+      <child link="link_grasp_center" />
   </joint>
   <!-- Gripper -->
