Commit message: wip: update robot inertia and weight

File: stretch_gazebo/urdf/stretch_main.xacro (robot description, xacro)
@@ -13,12 +13,19 @@
         rpy="0 0 0" />
       <mass
-        value="1.1912" />
-      <inertia
-        ixx="0.0034667"
-        ixy="-5.0568E-06"
-        ixz="0.00042861"
-        iyy="0.0052744"
-        iyz="-5.766E-05"
-        izz="0.0047945" />
+        value="50.1912" />
+        <inertia
+          ixx="0.8333"
+          ixy="0"
+          ixz="0"
+          iyy="1.2083"
+          iyz="0"
+          izz="1.7083"/>
+      <!-- <inertia -->
+      <!--   ixx="0.0034667" -->
+      <!--   ixy="-5.0568E-06" -->
+      <!--   ixz="0.00042861" -->
+      <!--   iyy="0.0052744" -->
+      <!--   iyz="-5.766E-05" -->
+      <!--   izz="0.0047945" /> -->
     </inertial>
     <visual>

File: stretch_gazebo/urdf/stretch_robotiq_gazebo.urdf.xacro (robot description, xacro)
@@ -504,5 +504,11 @@
       xyz="0 0 0" />
   </joint>
-  <link name="link_grasp_center" />
+  <link name="link_grasp_center">
+  <!--   <inertial> -->
+  <!--   <mass value="0"/> -->
+  <!--   <origin xyz="0 0 0" rpy="0 0 0"/> -->
+  <!--   <inertia ixx="0" iyy="0" izz="0" ixy="0" ixz="0" iyz="0"/> -->
+  <!-- </inertial>> -->
+  </link>
   <joint name="joint_grasp_center" type="fixed">
       <origin rpy="0 0 0" xyz="0 0 0.2" />

Commit message: wip: update center of gravity

File: stretch_gazebo/urdf/stretch_main.xacro (robot description, xacro)
@@ -9,6 +9,7 @@
     name="base_link">
     <inertial>
-      <origin
-        xyz="-0.11587 0.0019426 0.093621"
+    <!-- xyz="-0.11587 0.0019426 0.093621" -->
+      <origin
+        xyz="-0.2 0 0.01"
         rpy="0 0 0" />
       <mass
